File: Keyboard.kicad_pcb (KiCad board)
At the start: 2 copper layers, 231.1 x 96.5 mm, 154 parts, among them Q1 BSS138, Q2 BSS138, SW1 SW_Kailh_1u, SW10 SW_Kailh_1u, SW11 SW_Kailh_1u, SW12 SW_Kailh_1u, SW13 SW_Kailh_1u, SW14 SW_Kailh_1u, SW15 SW_Kailh_1u, SW16 SW_Kailh_1u, SW17 SW_Kailh_1u, SW18 SW_Kailh_1u, SW19 SW_Kailh_1u, SW2 SW_Kailh_1u, SW20 SW_Kailh_1u, SW21 SW_Kailh_1u, SW22 SW_Kailh_1u, SW23 SW_Kailh_1u, SW23_3u1 SW_Kailh_3u, SW24 SW_Kailh_1u, SW25 SW_Kailh_1u, SW26 SW_Kailh_1u, SW27 SW_Kailh_1u, SW28 SW_Kailh_1u, SW29 SW_Kailh_1u, SW3 SW_Kailh_1u, SW30 SW_Kailh_1u, SW31 SW_Kailh_1u, SW32 SW_Kailh_1u, SW33 SW_Kailh_1u, SW34 SW_Kailh_1u, SW35 SW_Kailh_1u, SW36 SW_Kailh_1u, SW37 SW_Kailh_1u, SW38 SW_Kailh_1u, SW39 SW_Kailh_1u, SW4 SW_Kailh_1u, SW40 SW_Kailh_1u, SW41 SW_Kailh_1u, SW42 SW_Kailh_1u, SW43 SW_Kailh_1u, SW44 SW_Kailh_1u, SW45 SW_Kailh_1u, SW5 SW_Kailh_1u, SW6 SW_Kailh_1u, SW7 SW_Kailh_1u, SW8 SW_Kailh_1u, SW9 SW_Kailh_1u, U1 PCAL6416APW, U2 Seeed Studio XIAO SAMD21, U3 NSI50350ADT4G

Commit message: finished pcb routing
Parts:
- removed RGB49, RGB50: ~, Keebio-Parts.pretty-master:SK6812-MINI-E
- added C1: 1uF, Capacitor_SMD:C_0805_2012Metric_Pad1.18x1.45mm_HandSolder, F.Cu at (238.8, 47.6)
- R1, R14, R15, R16: moved to B.Cu
- moved R1 351.3 mm to (248.0, 45.0)
- moved BT1 341.2 mm to (245.5, 41.5), turned to 90 degrees
- moved R14 333.9 mm to (230.6, 50.4), turned to 90 degrees
- moved R16 330.7 mm to (226.8, 44.3), turned to -90 degrees
- moved R15 329.8 mm to (226.6, 54.7), turned to 90 degrees
- moved U1 302.2 mm to (245.9, 52.3), turned to 180 degrees
- moved R17 225.6 mm to (213.2, 44.8), turned to 180 degrees
- moved Q2 225.5 mm to (207.9, 49.3), turned to 180 degrees
- moved R18 225.1 mm to (213.2, 42.0)
- moved Q1 223.4 mm to (205.8, 44.3), turned to -90 degrees
- moved U3 216.0 mm to (198.8, 55.6), turned to 90 degrees
- moved U2 21.4 mm to (227.4, 49.8)
Connections:
- BT1 pad 2: Net-(BT1--) -> GND
- RGB48 pad 2: Net-(RGB48-DOUT) -> unconnected-(RGB48-DOUT-Pad2)
- U1 pad 10: COL 2 -> LINE 2
- U1 pad 11: COL 1 -> LINE 1
- U1 pad 13: COL 5 -> COL 12
- U1 pad 14: COL 6 -> COL 11
- U1 pad 15: COL 7 -> COL 10
- U1 pad 16: COL 8 -> COL 9
- U1 pad 17: COL 9 -> COL 8
- U1 pad 18: COL 10 -> COL 7
- U1 pad 19: COL 11 -> COL 6
- U1 pad 20: COL 12 -> COL 5
- U1 pad 4: LINE 1 -> COL 1
- U1 pad 5: LINE 2 -> COL 2
- U1 pad 6: LINE 3 -> COL 3
- U1 pad 7: LINE 4 -> COL 4
- U1 pad 8: COL 4 -> LINE 4
- U1 pad 9: COL 3 -> LINE 3
- U2 pad 21: Net-(BT1--) -> unconnected-(U2-BAT--Pad21)
Routing:
- net Net-(RGB1-VDD): track 205.8 -> 1420.4 mm, vias 0 -> 49
- net GND: track 122.9 -> 1067.5 mm, vias 0 -> 16
- net COL 1: track 0.00 -> 375.3 mm, vias 0 -> 2
- net COL 2: track 0.00 -> 356.9 mm
- net LINE 4: track 0.00 -> 354.0 mm, vias 0 -> 11
- net LINE 3: track 0.00 -> 338.7 mm, vias 0 -> 13
- net COL 3: track 0.00 -> 335.4 mm
- net LINE 2: track 0.00 -> 318.7 mm, vias 0 -> 13
- net LINE 1: track 0.00 -> 279.3 mm, vias 0 -> 13
- net COL 4: track 0.00 -> 274.1 mm, vias 0 -> 2
- net COL 6: track 0.00 -> 200.8 mm, vias 0 -> 2
- net COL 5: track 0.00 -> 199.5 mm, vias 0 -> 2
- net COL 7: track 0.00 -> 159.2 mm, vias 0 -> 2
- net COL 8: track 0.00 -> 156.2 mm
- net COL 9: track 0.00 -> 133.6 mm
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Other:
- board size 231.1 x 96.5 mm -> 231.8 x 98.9 mm
